Commit message: cleanup plugins which are NA
Laser, UR5, and kinect removed.  Remove use of shell script in favor of package find. Build but  not running.

File: microtrac_gazebo/urdf/description.gazebo.xacro (robot description, xacro)
@@ -22,7 +22,4 @@
 -->
 <robot name="microtrac_robot_gazebo" xmlns:xacro="http://ros.org/wiki/xacro">
-  <xacro:arg name="laser_enabled" default="true" />
-  <xacro:arg name="ur5_enabled" default="false" />
-  <xacro:arg name="kinect_enabled" default="false" />
   <xacro:include filename="$(find microtrac_description)/urdf/microtrac.urdf.xacro" />
   <xacro:include filename="$(find microtrac_gazebo)/urdf/microtrac.gazebo.xacro" />
@@ -33,5 +30,5 @@
     </plugin>
   </gazebo>
-  <xacro:microtrac_robot />
+<!--  <xacro:microtrac_robot />-->
   <xacro:microtrac_robot_gazebo />
 </robot>

File: microtrac_gazebo/urdf/microtrac.gazebo.xacro (robot description, xacro)
@@ -22,5 +22,4 @@
 -->
 <robot name="microtrac_robot_gazebo" xmlns:xacro="http://ros.org/wiki/xacro">
-  <xacro:include filename="$(find microtrac_gazebo)/urdf/accessories/kinect_camera.gazebo.xacro"/>
   <xacro:macro name="microtrac_robot_gazebo">
     <gazebo>
@@ -53,31 +52,4 @@
       </plugin>
     </gazebo>
-    <xacro:if value="$(arg ur5_enabled)">
-      <!--Remove when https://github.com/ros-industrial/universal_robot/pull/168 is resolved -->
-      <gazebo reference="ur5_arm_shoulder_link">
-        <selfCollide>true</selfCollide>
-      </gazebo>
-      <gazebo reference="ur5_arm_upper_arm_link">
-        <selfCollide>true</selfCollide>
-      </gazebo>
-      <gazebo reference="ur5_arm_forearm_link">
-        <selfCollide>true</selfCollide>
-      </gazebo>
-      <gazebo reference="ur5_arm_wrist_1_link">
-        <selfCollide>true</selfCollide>
-      </gazebo>
-      <gazebo reference="ur5_arm_wrist_3_link">
-       <selfCollide>true</selfCollide>
-      </gazebo>
-      <gazebo reference="ur5_arm_wrist_2_link">
-        <selfCollide>true</selfCollide>
-      </gazebo>
-      <gazebo reference="ur5_arm_ee_link">
-        <selfCollide>true</selfCollide>
-      </gazebo>
-    </xacro:if>
-    <xacro:if value="$(arg kinect_enabled)">
-      <xacro:kinect_camera_gazebo prefix="camera"/>
-    </xacro:if>
-  </xacro:macro>
+</xacro:macro>
 </robot>
